Commit message: added IMU and localization part, added csv files for track building

File: psd_ws/src/psd_vehicle_description/urdf/materials.xacro (robot description, xacro)
@@ -44,6 +44,6 @@
     <elasticity>
       <ode>
-        <epsilon>0.8</epsilon> <!-- Coefficient of restitution (elasticity) -->
-        <kp>100000000.0</kp> <!-- Contact stiffness -->
+        <epsilon>0.01</epsilon> <!-- Coefficient of restitution (elasticity) -->
+        <kp>1000000.0</kp> <!-- Contact stiffness -->
         <kd>10.0</kd> <!-- Contact damping -->
       </ode>

File: psd_ws/src/psd_vehicle_description/urdf/psd_vehicle.urdf.xacro (robot description, xacro)
@@ -3,12 +3,15 @@
   <xacro:include filename="$(find psd_vehicle_description)/urdf/psd_vehicle_macro.urdf.xacro"/>
   <xacro:include filename="$(find psd_vehicle_description)/urdf/psd_vehicle_macro.ros2_control.xacro"/>
+  <xacro:property name="PI" value="3.14159265359" />
+  <xacro:property name="rot90" value="${90 * PI / 180}" />
   <!-- Load robot's macro with parameters -->
   <link name="home" />
   <!-- set prefix if multiple robots are used -->
   <xacro:psd_vehicle parent="home" >
-    <origin xyz="0 0 0.095" rpy="0 0 0" />          <!-- position robot in the world -->
+    <origin xyz="0 0 0.095" rpy="0 0 -${rot90}" />          <!-- position robot in the world -->
   </xacro:psd_vehicle>
   <xacro:psd_vehicle_ros2_control
     name="psd_vehicle"
   />
+  <xacro:include filename="$(find psd_vehicle_description)/urdf/imu.xacro"/>
 </robot>

File: psd_ws/src/psd_vehicle_description/urdf/psd_vehicle_macro.ros2_control.xacro (robot description, xacro)
@@ -69,4 +69,24 @@
       </joint>
     </ros2_control>
+     <!-- IMU sensor-->
+    <ros2_control name='IMU' type='sensor'>
+      <hardware>
+        <plugin>imu_sensor_broadcaster/IMUSensorBroadcaster</plugin>
+          <param name='sensor_name'>imu_sample</param>
+          <param name='frame_id'>imu_link</param>
+      </hardware>
+      <sensor name='imu_sample'>
+        <state_interface name='orientation.x'/>
+        <state_interface name='orientation.y'/>
+        <state_interface name='orientation.z'/>
+        <state_interface name='orientation.w'/>
+        <state_interface name='angular_velocity.x'/>
+        <state_interface name='angular_velocity.y'/>
+        <state_interface name='angular_velocity.z'/>
+        <state_interface name='linear_acceleration.x'/>
+        <state_interface name='linear_acceleration.y'/>
+        <state_interface name='linear_acceleration.z'/>
+      </sensor>
+    </ros2_control>
     <gazebo>
       <!-- Joint state publisher -->

File: psd_ws/src/psd_vehicle_description/urdf/psd_vehicle_macro.urdf.xacro (robot description, xacro)
@@ -237,4 +237,11 @@
       xyz="0.0 0.0 0.2"
       rpy="0.0 0.0 ${rot90}" />
+    <!-- position/odom -->
+    <link name="base_footprint"/>
+    <joint name="footprint_joint" type="fixed">
+      <parent link="chassis"/>
+      <child link="base_footprint"/>
+      <origin xyz="0.0 0.0 0.0" rpy="0 0 0"/>
+    </joint>
   </xacro:macro>
 </robot>
